File: KiCAD10/IR.kicad_sch (KiCad schematic)
At the start: 53 parts, among them SW1 RESET, SW2 SINGLE, SW3 SELECT, U10 74HC161, U11 SST39SF010 LSB, U12 74HC32, U35 74HC00, U36 ATmega328P, U6 74HC161, U7 SST39SF010 HSB, U8 74HC377, U9 SST39SF010 MSB, Y1 16MHz

Commit message: Add orderable MPNs for flash/RAM/MCU and document chip programming
- BOM.csv: add MPN column; specify PDIP package variants
  (SST39SF010A-70-4C-PHE, AS6C1008-55PCN, ATMEGA328P-PU) so the
  orderable part is unambiguous from the DIP-32/DIP-28 footprints.
- Store matching MPN properties on the U7/U9/U11/U15/U17/U36 symbols
  in the KiCad 10 schematic so they survive BOM regeneration.
- CLAUDE.md: document chip identification by silkscreen U-number,
  the package-suffix gotcha, and that U36 (ATmega) has no on-board
  ISP path and must be programmed off-board (DIP-socket Uno / ZIF).

Co-Authored-By: Claude Opus 4.8 (1M context) <noreply@anthropic.com>
Parts:
- U11, U7, U9: MPN (none) -> SST39SF010A-70-4C-PHE
- U36: MPN (none) -> ATMEGA328P-PU
Changed lines of the file:
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@@
 			)
 		)
+		(property "MPN" "ATMEGA328P-PU"
+			(at 34.036 66.04 0)
+			(hide yes)
+			(show_name no)
+			(do_not_autoplace no)
+			(effects
+				(font
+					(size 1.27 1.27)
+				)
+			)
+		)
 		(property "Value" "ATmega328P"
 			(at 34.036 66.04 0)
@@
 			)
 		)
+		(property "MPN" "SST39SF010A-70-4C-PHE"
+			(at 153.035 38.1 90)
+			(hide yes)
+			(show_name no)
+			(do_not_autoplace no)
+			(effects
+				(font
+					(size 1.27 1.27)
+				)
+			)
+		)
 		(property "Value" "SST39SF010 HSB"
 			(at 153.035 38.1 90)
@@
 			)
 		)
+		(property "MPN" "SST39SF010A-70-4C-PHE"
+			(at 198.755 38.1 90)
+			(hide yes)
+			(show_name no)
+			(do_not_autoplace no)
+			(effects
+				(font
+					(size 1.27 1.27)
+				)
+			)
+		)
 		(property "Value" "SST39SF010 MSB"
 			(at 198.755 38.1 90)
@@
 			)
 		)
+		(property "MPN" "SST39SF010A-70-4C-PHE"
+			(at 245.745 38.1 90)
+			(hide yes)
+			(show_name no)
+			(do_not_autoplace no)
+			(effects
+				(font
+					(size 1.27 1.27)
+				)
+			)
+		)

Commit message: Capture as-built LED colours as schematic Color field
Prepping the BOM/PCB for a prototype fab run: the front-panel LED
colour was only recorded per-footprint on the PCB (the Description
field, e.g. "LED GREEN, 2000mcd, 60°") and so never reached the
schematic-generated BOM. Copy that colour onto all 98 LED symbols as
a hidden `Color` property, matched by reference designator, so it
travels with the BOM the same way `MPN` does (add `Color` to the BOM
export field list). As-built distribution: Green 75, Yellow 11,
Red 7, White 4, Blue 1.

Source of truth for colour is now the schematic `Color` field; the
PCB footprint `Description` is the independent original and KiCad does
not auto-sync the two.

Also folds in KiCad 10 file normalisation that appeared on opening the
project (new .kicad_pro design-setting defaults; empty "element"
properties added to symbols on the top sheet). Document all of the
above in CLAUDE.md.

Co-Authored-By: Claude Opus 4.8 (1M context) <noreply@anthropic.com>
Parts:
- D1, D2, D3: Color (none) -> Green; element14 (none) -> 1581137
- D100: Color (none) -> Green
- D60, D61, D62, D63, D64, D67, D68, D69, D70, D71, D72, D73, D74, D75: Color (none) -> Green; element14 (none) -> 1003234
- D82, D87, D89, D90, D91: Color (none) -> Yellow
- U36: element14 (none) -> 1715487
- Y1: element14 (none) -> 1701139

Commit message: Normalise D1-D3 LED value case (LED_small -> LED_Small)
D1-D3 carried Value 'LED_small' (lowercase s) while every other
generic LED used 'LED_Small'. BOM grouping is case-sensitive, so the
typo split D1-D3 into their own line despite being the identical part.
Normalise the three so they merge with the main green LED group.

Co-Authored-By: Claude Opus 4.8 (1M context) <noreply@anthropic.com>
Parts:
- D1, D2, D3: value LED_small -> LED_Small
Changed lines of the file:
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@@
 			)
 		)
-		(property "Value" "LED_small"
+		(property "Value" "LED_Small"
 			(at 60.8965 60.96 0)
 			(hide yes)
@@
 			)
 		)
-		(property "Value" "LED_small"
+		(property "Value" "LED_Small"
 			(at 60.8965 53.34 0)
 			(hide yes)
@@
 			)
 		)
-		(property "Value" "LED_small"
+		(property "Value" "LED_Small"
 			(at 60.8965 57.15 0)
 			(hide yes)

Commit message: Tag green LEDs with Kingbright MPN L-53SGC
Green LED part is Kingbright L-53SGC — a manufacturer part number, so
it goes in MPN (all 75 green LEDs), unlike the red LEDs' Farnell code
which lives in Supplier Ref. Update the LED sourcing table in CLAUDE.md.

Co-Authored-By: Claude Opus 4.8 (1M context) <noreply@anthropic.com>
Parts:
- D1, D100, D2, D3, D60, D61, D62, D63, D64, D67, D68, D69, D70, D71, D72, D73, D74, D75: MPN (none) -> L-53SGC
Changed lines of the file:
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@@
 			)
 		)
+		(property "MPN" "L-53SGC"
+			(at 207.264 138.43 0)
+			(hide yes)
+			(show_name no)
+			(do_not_autoplace no)
+			(effects
+				(font
+					(size 1.27 1.27)
+				)
+			)
+		)
 		(property "Value" "LED_Small"
 			(at 205.74 138.3665 0)
@@
 			)
 		)
+		(property "MPN" "L-53SGC"
+			(at 199.644 138.43 0)
+			(hide yes)
+			(show_name no)
+			(do_not_autoplace no)
+			(effects
+				(font
+					(size 1.27 1.27)
+				)
+			)
+		)
 		(property "Value" "LED_Small"
 			(at 198.12 138.3665 0)
@@
 			)
 		)
+		(property "MPN" "L-53SGC"
+			(at 209.804 138.43 0)
+			(hide yes)
+			(show_name no)
+			(do_not_autoplace no)
+			(effects
+				(font
+					(size 1.27 1.27)
+				)
+			)
+		)
 		(property "Value" "LED_Small"
 			(at 208.28 138.3665 0)
@@
 			)
 		)
+		(property "MPN" "L-53SGC"
+			(at 254.254 137.16 0)
+			(hide yes)
+			(show_name no)
+			(do_not_autoplace no)
+			(effects
+				(font
+					(size 1.27 1.27)
+				)
+			)
+		)
 		(property "Value" "LED_Small"
 			(at 252.73 137.0965 0)
@@
 			)
 		)
+		(property "MPN" "L-53SGC"
+			(at 202.184 138.43 0)
+			(hide yes)
+			(show_name no)
+			(do_not_autoplace no)
+			(effects
+				(font
+					(size 1.27 1.27)
+				)
+			)
+		)
 		(property "Value" "LED_Small"
 			(at 200.66 138.3665 0)
@@
 			)
 		)
+		(property "MPN" "L-53SGC"
+			(at 113.284 67.31 0)
+			(hide yes)
+			(show_name no)
+			(do_not_autoplace no)
+			(effects
+				(font
+					(size 1.27 1.27)
+				)
+			)
+		)
 		(property "Value" "CLK"
 			(at 112.268 67.31 0)
@@
 			)
 		)
+		(property "MPN" "L-53SGC"
+			(at 161.544 138.43 0)
+			(hide yes)
+			(show_name no)
+			(do_not_autoplace no)
+			(effects
+				(font
+					(size 1.27 1.27)
+				)
+			)
+		)
 		(property "Value" "LED_Small"
 			(at 160.02 138.3665 0)
@@
 			)
 		)
+		(property "MPN" "L-53SGC"
+			(at 249.174 137.16 0)
+			(hide yes)
+			(show_name no)
+			(do_not_autoplace no)
+			(effects
+				(font
+					(size 1.27 1.27)
+				)
+			)
+		)
 		(property "Value" "LED_Small"
 			(at 247.65 137.0965 0)
@@
 			)
 		)
+		(property "MPN" "L-53SGC"
+			(at 204.724 138.43 0)
+			(hide yes)
+			(show_name no)
+			(do_not_autoplace no)
+			(effects
+				(font
+					(size 1.27 1.27)
+				)
+			)
+		)
 		(property "Value" "LED_Small"
 			(at 203.2 138.3665 0)
@@
 			)
 		)
+		(property "MPN" "L-53SGC"
+			(at 212.344 138.43 0)
+			(hide yes)
+			(show_name no)
+			(do_not_autoplace no)
+			(effects
+				(font
+					(size 1.27 1.27)
+				)
+			)
+		)
 		(property "Value" "LED_Small"
 			(at 210.82 138.3665 0)
@@
 			)
 		)
+		(property "MPN" "L-53SGC"
+			(at 159.004 138.43 0)
+			(hide yes)
+			(show_name no)
+			(do_not_autoplace no)
+			(effects
+				(font
+					(size 1.27 1.27)
+				)
+			)
+		)
 		(property "Value" "LED_Small"
 			(at 157.48 138.3665 0)
@@
 			)
 		)
+		(property "MPN" "L-53SGC"
+			(at 60.96 62.484 0)
+			(hide yes)
+			(show_name no)
+			(do_not_autoplace no)
+			(effects
+				(font
+					(size 1.27 1.27)
+				)
+			)
+		)
 		(property "Value" "LED_Small"
 			(at 60.8965 60.96 0)
@@
 			)
 		)
+		(property "MPN" "L-53SGC"
+			(at 246.634 137.16 0)
+			(hide yes)
+			(show_name no)
+			(do_not_autoplace no)
+			(effects
+				(font
+					(size 1.27 1.27)
+				)
+			)
+		)
 		(property "Value" "LED_Small"
 			(at 245.11 137.0965 0)
@@
 			)
 		)
+		(property "MPN" "L-53SGC"
+			(at 60.96 54.864 0)
+			(hide yes)
+			(show_name no)
+			(do_not_autoplace no)
+			(effects
+				(font
+					(size 1.27 1.27)
+				)
+			)
+		)
 		(property "Value" "LED_Small"
 			(at 60.8965 53.34 0)
@@
 			)
 		)
+		(property "MPN" "L-53SGC"
+			(at 156.464 138.43 0)
+			(hide yes)
+			(show_name no)
+			(do_not_autoplace no)
+			(effects
+				(font
+					(size 1.27 1.27)
+				)
+			)
+		)
 		(property "Value" "LED_Small"
 			(at 154.94 138.3665 0)
@@
 			)
 		)
+		(property "MPN" "L-53SGC"
+			(at 251.714 137.16 0)
+			(hide yes)
+			(show_name no)
+			(do_not_autoplace no)
+			(effects
+				(font
+					(size 1.27 1.27)
+				)
+			)
+		)
 		(property "Value" "LED_Small"
 			(at 250.19 137.0965 0)
@@
 			)
 		)
+		(property "MPN" "L-53SGC"
+			(at 153.924 138.43 0)
+			(hide yes)
+			(show_name no)
+			(do_not_autoplace no)
+			(effects
+				(font
+					(size 1.27 1.27)
+				)
+			)
+		)
 		(property "Value" "LED_Small"
 			(at 152.4 138.3665 0)
@@
 			(at 60.96 58.674 0)
 			(hide yes)
+			(show_name no)
+			(do_not_autoplace no)
+			(effects
+				(font
+					(size 1.27 1.27)
+				)
+			)
+		)
+		(property "MPN" "L-53SGC"
+			(at 60.96 58.674 0)
+			(hide yes)

Commit message: Standardise LEDs on Supplier Ref (Element14-only sourcing)
Only Element14 is used for LEDs, so identify every LED by its
Element14 Supplier Ref and carry no MPN on LEDs. Move the green LEDs'
L-53SGC from MPN to Supplier Ref (red 703-0100 already there). MPN
stays reserved for the socketed chips (manufacturer parts). Update the
LED sourcing table in CLAUDE.md.

Co-Authored-By: Claude Opus 4.8 (1M context) <noreply@anthropic.com>
Parts:
- D1, D100, D2, D3, D60, D61, D62, D63, D64, D67, D68, D69, D70, D71, D72, D73, D74, D75: MPN L-53SGC -> (none); Supplier Ref (none) -> L-53SGC
Changed lines of the file:
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@@
 			)
 		)
-		(property "MPN" "L-53SGC"
+		(property "Supplier Ref" "L-53SGC"
 			(at 207.264 138.43 0)
 			(hide yes)
@@
 			)
 		)
-		(property "MPN" "L-53SGC"
+		(property "Supplier Ref" "L-53SGC"
 			(at 199.644 138.43 0)
 			(hide yes)
@@
 			)
 		)
-		(property "MPN" "L-53SGC"
+		(property "Supplier Ref" "L-53SGC"
 			(at 209.804 138.43 0)
 			(hide yes)
@@
 			)
 		)
-		(property "MPN" "L-53SGC"
+		(property "Supplier Ref" "L-53SGC"
 			(at 254.254 137.16 0)
 			(hide yes)
@@
 			)
 		)
-		(property "MPN" "L-53SGC"
+		(property "Supplier Ref" "L-53SGC"
 			(at 202.184 138.43 0)
 			(hide yes)
@@
 			)
 		)
-		(property "MPN" "L-53SGC"
+		(property "Supplier Ref" "L-53SGC"
 			(at 113.284 67.31 0)
 			(hide yes)
@@
 			)
 		)
-		(property "MPN" "L-53SGC"
+		(property "Supplier Ref" "L-53SGC"
 			(at 161.544 138.43 0)
 			(hide yes)
@@
 			)
 		)
-		(property "MPN" "L-53SGC"
+		(property "Supplier Ref" "L-53SGC"
 			(at 249.174 137.16 0)
 			(hide yes)
@@
 			)
 		)
-		(property "MPN" "L-53SGC"
+		(property "Supplier Ref" "L-53SGC"
 			(at 204.724 138.43 0)
 			(hide yes)
@@
 			)
 		)
-		(property "MPN" "L-53SGC"
+		(property "Supplier Ref" "L-53SGC"
 			(at 212.344 138.43 0)
 			(hide yes)
@@
 			)
 		)
-		(property "MPN" "L-53SGC"
+		(property "Supplier Ref" "L-53SGC"
 			(at 159.004 138.43 0)
 			(hide yes)
@@
 			)
 		)
-		(property "MPN" "L-53SGC"
+		(property "Supplier Ref" "L-53SGC"
 			(at 60.96 62.484 0)
 			(hide yes)
@@
 			)
 		)
-		(property "MPN" "L-53SGC"
+		(property "Supplier Ref" "L-53SGC"
 			(at 246.634 137.16 0)
 			(hide yes)
@@
 			)
 		)
-		(property "MPN" "L-53SGC"
+		(property "Supplier Ref" "L-53SGC"
 			(at 60.96 54.864 0)
 			(hide yes)
@@
 			)
 		)
-		(property "MPN" "L-53SGC"
+		(property "Supplier Ref" "L-53SGC"
 			(at 156.464 138.43 0)
 			(hide yes)
@@
 			)
 		)
-		(property "MPN" "L-53SGC"
+		(property "Supplier Ref" "L-53SGC"
 			(at 251.714 137.16 0)
 			(hide yes)
@@
 			)
 		)
-		(property "MPN" "L-53SGC"
+		(property "Supplier Ref" "L-53SGC"
 			(at 153.924 138.43 0)
 			(hide yes)
@@
 			)
 		)
-		(property "MPN" "L-53SGC"
+		(property "Supplier Ref" "L-53SGC"
 			(at 60.96 58.674 0)
 			(hide yes)

Commit message: Tag yellow LEDs with Element14 Supplier Ref MCL053YD
Add Supplier Ref MCL053YD to the 11 yellow front-panel LEDs and update
the LED sourcing table in CLAUDE.md. White and blue still uncoded.

Co-Authored-By: Claude Opus 4.8 (1M context) <noreply@anthropic.com>
Parts:
- D82, D87, D89, D90, D91: Supplier Ref (none) -> MCL053YD
Changed lines of the file:
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@@
 			)
 		)
+		(property "Supplier Ref" "MCL053YD"
+			(at 127.254 67.31 0)
+			(hide yes)
+			(show_name no)
+			(do_not_autoplace no)
+			(effects
+				(font
+					(size 1.27 1.27)
+				)
+			)
+		)
 		(property "Value" "TI"
 			(at 127.254 67.31 0)
@@
 			)
 		)
+		(property "Supplier Ref" "MCL053YD"
+			(at 120.904 93.98 0)
+			(hide yes)
+			(show_name no)
+			(do_not_autoplace no)
+			(effects
+				(font
+					(size 1.27 1.27)
+				)
+			)
+		)
 		(property "Value" "II"
 			(at 121.158 93.98 0)
@@
 			)
 		)
+		(property "Supplier Ref" "MCL053YD"
+			(at 113.284 93.98 0)
+			(hide yes)
+			(show_name no)
+			(do_not_autoplace no)
+			(effects
+				(font
+					(size 1.27 1.27)
+				)
+			)
+		)
 		(property "Value" "FI"
 			(at 113.538 93.98 0)
@@
 			)
 		)
+		(property "Supplier Ref" "MCL053YD"
+			(at 128.524 93.98 0)
+			(hide yes)
+			(show_name no)
+			(do_not_autoplace no)
+			(effects
+				(font
+					(size 1.27 1.27)
+				)
+			)
+		)
 		(property "Value" "IC"
 			(at 128.524 93.98 0)
@@
 			(at 120.904 67.31 0)
 			(hide yes)
+			(show_name no)
+			(do_not_autoplace no)
+			(effects
+				(font
+					(size 1.27 1.27)
+				)
+			)
+		)
+		(property "Supplier Ref" "MCL053YD"
+			(at 120.904 67.31 0)
+			(hide yes)
