File: KiCAD10/RAM.kicad_sch (KiCad schematic)
At the start: 32 parts, among them U14 74HC161, U15 SST39SF010 SSD, U16 74HC161, U17 AS6C1008 RAM, U18 74HC161, U19 74HC161

Commit message: Add orderable MPNs for flash/RAM/MCU and document chip programming
- BOM.csv: add MPN column; specify PDIP package variants
  (SST39SF010A-70-4C-PHE, AS6C1008-55PCN, ATMEGA328P-PU) so the
  orderable part is unambiguous from the DIP-32/DIP-28 footprints.
- Store matching MPN properties on the U7/U9/U11/U15/U17/U36 symbols
  in the KiCad 10 schematic so they survive BOM regeneration.
- CLAUDE.md: document chip identification by silkscreen U-number,
  the package-suffix gotcha, and that U36 (ATmega) has no on-board
  ISP path and must be programmed off-board (DIP-socket Uno / ZIF).

Co-Authored-By: Claude Opus 4.8 (1M context) <noreply@anthropic.com>
Parts:
- U15: MPN (none) -> SST39SF010A-70-4C-PHE
- U17: MPN (none) -> AS6C1008-55PCN
Changed lines of the file:
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@@
+			)
+		)
+		(property "MPN" "AS6C1008-55PCN"
+			(at 172.72 39.37 90)
+			(hide yes)
+			(show_name no)
+			(do_not_autoplace no)
+			(effects
+				(font
+					(size 1.27 1.27)
+				)
 			)
 		)
@@
 			)
 		)
+		(property "MPN" "SST39SF010A-70-4C-PHE"
+			(at 110.49 39.37 90)
+			(hide yes)
+			(show_name no)
+			(do_not_autoplace no)
+			(effects
+				(font
+					(size 1.27 1.27)
+				)
+			)
+		)

Commit message: Capture as-built LED colours as schematic Color field
Prepping the BOM/PCB for a prototype fab run: the front-panel LED
colour was only recorded per-footprint on the PCB (the Description
field, e.g. "LED GREEN, 2000mcd, 60°") and so never reached the
schematic-generated BOM. Copy that colour onto all 98 LED symbols as
a hidden `Color` property, matched by reference designator, so it
travels with the BOM the same way `MPN` does (add `Color` to the BOM
export field list). As-built distribution: Green 75, Yellow 11,
Red 7, White 4, Blue 1.

Source of truth for colour is now the schematic `Color` field; the
PCB footprint `Description` is the independent original and KiCad does
not auto-sync the two.

Also folds in KiCad 10 file normalisation that appeared on opening the
project (new .kicad_pro design-setting defaults; empty "element"
properties added to symbols on the top sheet). Document all of the
above in CLAUDE.md.

Co-Authored-By: Claude Opus 4.8 (1M context) <noreply@anthropic.com>
Parts:
- D10, D11, D12, D13, D14, D15, D16, D17, D18, D19, D4, D5, D6, D7, D8, D9: Color (none) -> Green; element14 (none) -> 1003234
- D85, D86: Color (none) -> Yellow
- D88: Color (none) -> White
- D99: Color (none) -> Red

Commit message: Tag red LEDs with Element14 order code 703-0100
Add MPN 703-0100 to the 7 red front-panel LEDs (D66 AO, D77 BO,
D78 EO, D80 TO, D81 COH, D83 COL, D99 RO) for the Element14 order.

Co-Authored-By: Claude Opus 4.8 (1M context) <noreply@anthropic.com>
Parts:
- D99: MPN (none) -> 703-0100
Changed lines of the file:
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@@
+			)
+		)
+		(property "MPN" "703-0100"
+			(at 134.874 132.08 0)
+			(hide yes)
+			(show_name no)
+			(do_not_autoplace no)
+			(effects
+				(font
+					(size 1.27 1.27)
+				)
 			)
 		)

Commit message: Move LED Element14 code from MPN to Supplier Ref field
Element14/Farnell order codes are distributor codes, not manufacturer
part numbers, so keep them out of MPN (which holds manufacturer PNs
like SST39SF010A-70-4C-PHE for the chips). Migrate the red LEDs'
703-0100 into a dedicated 'Supplier Ref' property and document the
MPN vs Supplier Ref convention in CLAUDE.md.

Co-Authored-By: Claude Opus 4.8 (1M context) <noreply@anthropic.com>
Parts:
- D99: MPN 703-0100 -> (none); Supplier Ref (none) -> 703-0100
Changed lines of the file:
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@@
 			)
 		)
-		(property "MPN" "703-0100"
+		(property "Supplier Ref" "703-0100"
 			(at 134.874 132.08 0)
 			(hide yes)

Commit message: Tag green LEDs with Kingbright MPN L-53SGC
Green LED part is Kingbright L-53SGC — a manufacturer part number, so
it goes in MPN (all 75 green LEDs), unlike the red LEDs' Farnell code
which lives in Supplier Ref. Update the LED sourcing table in CLAUDE.md.

Co-Authored-By: Claude Opus 4.8 (1M context) <noreply@anthropic.com>
Parts:
- D10, D11, D12, D13, D14, D15, D16, D17, D18, D19, D4, D5, D6, D7, D8, D9: MPN (none) -> L-53SGC
Changed lines of the file:
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@@
 			)
 		)
+		(property "MPN" "L-53SGC"
+			(at 103.886 132.08 0)
+			(hide yes)
+			(show_name no)
+			(do_not_autoplace no)
+			(effects
+				(font
+					(size 1.27 1.27)
+				)
+			)
+		)
 		(property "Value" "LED_Small"
 			(at 105.41 132.0165 0)
@@
 			)
 		)
+		(property "MPN" "L-53SGC"
+			(at 197.866 132.08 0)
+			(hide yes)
+			(show_name no)
+			(do_not_autoplace no)
+			(effects
+				(font
+					(size 1.27 1.27)
+				)
+			)
+		)
 		(property "Value" "LED_Small"
 			(at 199.39 132.0165 0)
@@
 			)
 		)
+		(property "MPN" "L-53SGC"
+			(at 210.566 132.08 0)
+			(hide yes)
+			(show_name no)
+			(do_not_autoplace no)
+			(effects
+				(font
+					(size 1.27 1.27)
+				)
+			)
+		)
 		(property "Value" "LED_Small"
 			(at 212.09 132.0165 0)
@@
 			)
 		)
+		(property "MPN" "L-53SGC"
+			(at 208.026 132.08 0)
+			(hide yes)
+			(show_name no)
+			(do_not_autoplace no)
+			(effects
+				(font
+					(size 1.27 1.27)
+				)
+			)
+		)
 		(property "Value" "LED_Small"
 			(at 209.55 132.0165 0)
@@
 			)
 		)
+		(property "MPN" "L-53SGC"
+			(at 101.346 132.08 0)
+			(hide yes)
+			(show_name no)
+			(do_not_autoplace no)
+			(effects
+				(font
+					(size 1.27 1.27)
+				)
+			)
+		)
 		(property "Value" "LED_Small"
 			(at 102.87 132.0165 0)
@@
 			)
 		)
+		(property "MPN" "L-53SGC"
+			(at 108.966 132.08 0)
+			(hide yes)
+			(show_name no)
+			(do_not_autoplace no)
+			(effects
+				(font
+					(size 1.27 1.27)
+				)
+			)
+		)
 		(property "Value" "LED_Small"
 			(at 110.49 132.0165 0)
@@
 			)
 		)
+		(property "MPN" "L-53SGC"
+			(at 96.266 132.08 0)
+			(hide yes)
+			(show_name no)
+			(do_not_autoplace no)
+			(effects
+				(font
+					(size 1.27 1.27)
+				)
+			)
+		)
 		(property "Value" "LED_Small"
 			(at 97.79 132.0165 0)
@@
 			)
 		)
+		(property "MPN" "L-53SGC"
+			(at 202.946 132.08 0)
+			(hide yes)
+			(show_name no)
+			(do_not_autoplace no)
+			(effects
+				(font
+					(size 1.27 1.27)
+				)
+			)
+		)
 		(property "Value" "LED_Small"
 			(at 204.47 132.0165 0)
@@
 			)
 		)
+		(property "MPN" "L-53SGC"
+			(at 213.106 132.08 0)
+			(hide yes)
+			(show_name no)
+			(do_not_autoplace no)
+			(effects
+				(font
+					(size 1.27 1.27)
+				)
+			)
+		)
 		(property "Value" "LED_Small"
 			(at 214.63 132.0165 0)
@@
 			)
 		)
+		(property "MPN" "L-53SGC"
+			(at 195.326 132.08 0)
+			(hide yes)
+			(show_name no)
+			(do_not_autoplace no)
+			(effects
+				(font
+					(size 1.27 1.27)
+				)
+			)
+		)
 		(property "Value" "LED_Small"
 			(at 196.85 132.0165 0)
@@
 			)
 		)
+		(property "MPN" "L-53SGC"
+			(at 200.406 132.08 0)
+			(hide yes)
+			(show_name no)
+			(do_not_autoplace no)
+			(effects
+				(font
+					(size 1.27 1.27)
+				)
+			)
+		)
 		(property "Value" "LED_Small"
 			(at 201.93 132.0165 0)
@@
 			)
 		)
+		(property "MPN" "L-53SGC"
+			(at 106.426 132.08 0)
+			(hide yes)
+			(show_name no)
+			(do_not_autoplace no)
+			(effects
+				(font
+					(size 1.27 1.27)
+				)
+			)
+		)
 		(property "Value" "LED_Small"
 			(at 107.95 132.0165 0)
@@
 			)
 		)
+		(property "MPN" "L-53SGC"
+			(at 93.726 132.08 0)
+			(hide yes)
+			(show_name no)
+			(do_not_autoplace no)
+			(effects
+				(font
+					(size 1.27 1.27)
+				)
+			)
+		)
 		(property "Value" "LED_Small"
 			(at 95.25 132.0165 0)
@@
 			)
 		)
+		(property "MPN" "L-53SGC"
+			(at 98.806 132.08 0)
+			(hide yes)
+			(show_name no)
+			(do_not_autoplace no)
+			(effects
+				(font
+					(size 1.27 1.27)
+				)
+			)
+		)
 		(property "Value" "LED_Small"
 			(at 100.33 132.0165 0)
@@
 			)
 		)
+		(property "MPN" "L-53SGC"
+			(at 205.486 132.08 0)
+			(hide yes)
+			(show_name no)
+			(do_not_autoplace no)
+			(effects
+				(font
+					(size 1.27 1.27)
+				)
+			)
+		)
 		(property "Value" "LED_Small"
 			(at 207.01 132.0165 0)
@@
 			(at 111.506 132.08 0)
 			(hide yes)
+			(show_name no)
+			(do_not_autoplace no)
+			(effects
+				(font
+					(size 1.27 1.27)
+				)
+			)
+		)
+		(property "MPN" "L-53SGC"
+			(at 111.506 132.08 0)
+			(hide yes)

Commit message: Standardise LEDs on Supplier Ref (Element14-only sourcing)
Only Element14 is used for LEDs, so identify every LED by its
Element14 Supplier Ref and carry no MPN on LEDs. Move the green LEDs'
L-53SGC from MPN to Supplier Ref (red 703-0100 already there). MPN
stays reserved for the socketed chips (manufacturer parts). Update the
LED sourcing table in CLAUDE.md.

Co-Authored-By: Claude Opus 4.8 (1M context) <noreply@anthropic.com>
Parts:
- D10, D11, D12, D13, D14, D15, D16, D17, D18, D19, D4, D5, D6, D7, D8, D9: MPN L-53SGC -> (none); Supplier Ref (none) -> L-53SGC
Changed lines of the file:
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@@
 			)
 		)
-		(property "MPN" "L-53SGC"
+		(property "Supplier Ref" "L-53SGC"
 			(at 103.886 132.08 0)
 			(hide yes)
@@
 			)
 		)
-		(property "MPN" "L-53SGC"
+		(property "Supplier Ref" "L-53SGC"
 			(at 197.866 132.08 0)
 			(hide yes)
@@
 			)
 		)
-		(property "MPN" "L-53SGC"
+		(property "Supplier Ref" "L-53SGC"
 			(at 210.566 132.08 0)
 			(hide yes)
@@
 			)
 		)
-		(property "MPN" "L-53SGC"
+		(property "Supplier Ref" "L-53SGC"
 			(at 208.026 132.08 0)
 			(hide yes)
@@
 			)
 		)
-		(property "MPN" "L-53SGC"
+		(property "Supplier Ref" "L-53SGC"
 			(at 101.346 132.08 0)
 			(hide yes)
@@
 			)
 		)
-		(property "MPN" "L-53SGC"
+		(property "Supplier Ref" "L-53SGC"
 			(at 108.966 132.08 0)
 			(hide yes)
@@
 			)
 		)
-		(property "MPN" "L-53SGC"
+		(property "Supplier Ref" "L-53SGC"
 			(at 96.266 132.08 0)
 			(hide yes)
@@
 			)
 		)
-		(property "MPN" "L-53SGC"
+		(property "Supplier Ref" "L-53SGC"
 			(at 202.946 132.08 0)
 			(hide yes)
@@
 			)
 		)
-		(property "MPN" "L-53SGC"
+		(property "Supplier Ref" "L-53SGC"
 			(at 213.106 132.08 0)
 			(hide yes)
@@
 			)
 		)
-		(property "MPN" "L-53SGC"
+		(property "Supplier Ref" "L-53SGC"
 			(at 195.326 132.08 0)
 			(hide yes)
@@
 			)
 		)
-		(property "MPN" "L-53SGC"
+		(property "Supplier Ref" "L-53SGC"
 			(at 200.406 132.08 0)
 			(hide yes)
@@
 			)
 		)
-		(property "MPN" "L-53SGC"
+		(property "Supplier Ref" "L-53SGC"
 			(at 106.426 132.08 0)
 			(hide yes)
@@
 			)
 		)
-		(property "MPN" "L-53SGC"
+		(property "Supplier Ref" "L-53SGC"
 			(at 93.726 132.08 0)
 			(hide yes)
@@
 			)
 		)
-		(property "MPN" "L-53SGC"
+		(property "Supplier Ref" "L-53SGC"
 			(at 98.806 132.08 0)
 			(hide yes)
@@
 			)
 		)
-		(property "MPN" "L-53SGC"
+		(property "Supplier Ref" "L-53SGC"
 			(at 205.486 132.08 0)
 			(hide yes)
@@
 			)
 		)
-		(property "MPN" "L-53SGC"
+		(property "Supplier Ref" "L-53SGC"
 			(at 111.506 132.08 0)
 			(hide yes)

Commit message: Tag yellow LEDs with Element14 Supplier Ref MCL053YD
Add Supplier Ref MCL053YD to the 11 yellow front-panel LEDs and update
the LED sourcing table in CLAUDE.md. White and blue still uncoded.

Co-Authored-By: Claude Opus 4.8 (1M context) <noreply@anthropic.com>
Parts:
- D85, D86: Supplier Ref (none) -> MCL053YD
Changed lines of the file:
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@@
+			)
+		)
+		(property "Supplier Ref" "MCL053YD"
+			(at 150.114 132.08 0)
+			(hide yes)
+			(show_name no)
+			(do_not_autoplace no)
+			(effects
+				(font
+					(size 1.27 1.27)
+				)
 			)
 		)
@@
 			(at 157.734 132.08 0)
 			(hide yes)
+			(show_name no)
+			(do_not_autoplace no)
+			(effects
+				(font
+					(size 1.27 1.27)
+				)
+			)
+		)
+		(property "Supplier Ref" "MCL053YD"
+			(at 157.734 132.08 0)
+			(hide yes)
