File: KiCAD10/RAM.kicad_sch (KiCad schematic)
At the start: 32 parts, among them U14 74HC161, U15 SST39SF010 SSD, U16 74HC161, U17 AS6C1008 RAM, U18 74HC161, U19 74HC161

Commit message: Tag white LEDs with Element14 Supplier Ref C512A-WNN-CZ0B0151
Add Supplier Ref C512A-WNN-CZ0B0151 to the 4 white front-panel LEDs
and update the LED sourcing table in CLAUDE.md. Only blue left.

Co-Authored-By: Claude Opus 4.8 (1M context) <noreply@anthropic.com>
Parts:
- D88: Supplier Ref (none) -> C512A-WNN-CZ0B0151
Changed lines of the file:
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@@
+			)
+		)
+		(property "Supplier Ref" "C512A-WNN-CZ0B0151"
+			(at 147.066 132.08 0)
+			(hide yes)
+			(show_name no)
+			(do_not_autoplace no)
+			(effects
+				(font
+					(size 1.27 1.27)
+				)
 			)
 		)

Commit message: Fix red LED Supplier Ref: use Element14 order code 2112111
703-0100 was the Multicomp MPN, not an Element14 order code. All 7
red LEDs (AO BO EO TO COH COL RO) now carry the numeric code, and
the CLAUDE.md sourcing table matches.

Co-Authored-By: Claude Fable 5 <noreply@anthropic.com>
Parts:
- D99: Supplier Ref 703-0100 -> 2112111
Changed lines of the file:
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@@
 			)
 		)
-		(property "Supplier Ref" "703-0100"
+		(property "Supplier Ref" "2112111"
 			(at 134.874 132.08 0)
 			(hide yes)
