File: KiCAD10/PC.kicad_sch (KiCad schematic)
At the start: 34 parts, among them U24 74HC245, U25 74HC161, U26 74HC161, U27 74HC245, U28 74HC161, U29 74HC161

Commit message: Capture as-built LED colours as schematic Color field
Prepping the BOM/PCB for a prototype fab run: the front-panel LED
colour was only recorded per-footprint on the PCB (the Description
field, e.g. "LED GREEN, 2000mcd, 60°") and so never reached the
schematic-generated BOM. Copy that colour onto all 98 LED symbols as
a hidden `Color` property, matched by reference designator, so it
travels with the BOM the same way `MPN` does (add `Color` to the BOM
export field list). As-built distribution: Green 75, Yellow 11,
Red 7, White 4, Blue 1.

Source of truth for colour is now the schematic `Color` field; the
PCB footprint `Description` is the independent original and KiCad does
not auto-sync the two.

Also folds in KiCad 10 file normalisation that appeared on opening the
project (new .kicad_pro design-setting defaults; empty "element"
properties added to symbols on the top sheet). Document all of the
above in CLAUDE.md.

Co-Authored-By: Claude Opus 4.8 (1M context) <noreply@anthropic.com>
Parts:
- D20, D21, D22, D23, D24, D25, D26, D27, D28, D29, D30, D31, D32, D33, D34, D35: Color (none) -> Green; element14 (none) -> 1003234
- D79, D84: Color (none) -> Yellow
- D81, D83: Color (none) -> Red
- D92: Color (none) -> White

Commit message: Tag red LEDs with Element14 order code 703-0100
Add MPN 703-0100 to the 7 red front-panel LEDs (D66 AO, D77 BO,
D78 EO, D80 TO, D81 COH, D83 COL, D99 RO) for the Element14 order.

Co-Authored-By: Claude Opus 4.8 (1M context) <noreply@anthropic.com>
Parts:
- D81, D83: MPN (none) -> 703-0100
Changed lines of the file:
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@@
+			)
+		)
+		(property "MPN" "703-0100"
+			(at 176.784 137.16 0)
+			(hide yes)
+			(show_name no)
+			(do_not_autoplace no)
+			(effects
+				(font
+					(size 1.27 1.27)
+				)
 			)
 		)
@@
 			(at 153.924 137.16 0)
 			(hide yes)
+			(show_name no)
+			(do_not_autoplace no)
+			(effects
+				(font
+					(size 1.27 1.27)
+				)
+			)
+		)
+		(property "MPN" "703-0100"
+			(at 153.924 137.16 0)
+			(hide yes)

Commit message: Move LED Element14 code from MPN to Supplier Ref field
Element14/Farnell order codes are distributor codes, not manufacturer
part numbers, so keep them out of MPN (which holds manufacturer PNs
like SST39SF010A-70-4C-PHE for the chips). Migrate the red LEDs'
703-0100 into a dedicated 'Supplier Ref' property and document the
MPN vs Supplier Ref convention in CLAUDE.md.

Co-Authored-By: Claude Opus 4.8 (1M context) <noreply@anthropic.com>
Parts:
- D81, D83: MPN 703-0100 -> (none); Supplier Ref (none) -> 703-0100
Changed lines of the file:
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@@
 			)
 		)
-		(property "MPN" "703-0100"
+		(property "Supplier Ref" "703-0100"
 			(at 176.784 137.16 0)
 			(hide yes)
@@
 			)
 		)
-		(property "MPN" "703-0100"
+		(property "Supplier Ref" "703-0100"
 			(at 153.924 137.16 0)
 			(hide yes)

Commit message: Tag green LEDs with Kingbright MPN L-53SGC
Green LED part is Kingbright L-53SGC — a manufacturer part number, so
it goes in MPN (all 75 green LEDs), unlike the red LEDs' Farnell code
which lives in Supplier Ref. Update the LED sourcing table in CLAUDE.md.

Co-Authored-By: Claude Opus 4.8 (1M context) <noreply@anthropic.com>
Parts:
- D20, D21, D22, D23, D24, D25, D26, D27, D28, D29, D30, D31, D32, D33, D34, D35: MPN (none) -> L-53SGC
Changed lines of the file:
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@@
 			)
 		)
+		(property "MPN" "L-53SGC"
+			(at 105.156 135.89 0)
+			(hide yes)
+			(show_name no)
+			(do_not_autoplace no)
+			(effects
+				(font
+					(size 1.27 1.27)
+				)
+			)
+		)
 		(property "Value" "LED_Small"
 			(at 106.68 135.8265 0)
@@
 			)
 		)
+		(property "MPN" "L-53SGC"
+			(at 238.506 137.16 0)
+			(hide yes)
+			(show_name no)
+			(do_not_autoplace no)
+			(effects
+				(font
+					(size 1.27 1.27)
+				)
+			)
+		)
 		(property "Value" "LED_Small"
 			(at 240.03 137.0965 0)
@@
 			)
 		)
+		(property "MPN" "L-53SGC"
+			(at 241.046 137.16 0)
+			(hide yes)
+			(show_name no)
+			(do_not_autoplace no)
+			(effects
+				(font
+					(size 1.27 1.27)
+				)
+			)
+		)
 		(property "Value" "LED_Small"
 			(at 242.57 137.0965 0)
@@
 			)
 		)
+		(property "MPN" "L-53SGC"
+			(at 243.586 137.16 0)
+			(hide yes)
+			(show_name no)
+			(do_not_autoplace no)
+			(effects
+				(font
+					(size 1.27 1.27)
+				)
+			)
+		)
 		(property "Value" "LED_Small"
 			(at 245.11 137.0965 0)
@@
 			)
 		)
+		(property "MPN" "L-53SGC"
+			(at 246.126 137.16 0)
+			(hide yes)
+			(show_name no)
+			(do_not_autoplace no)
+			(effects
+				(font
+					(size 1.27 1.27)
+				)
+			)
+		)
 		(property "Value" "LED_Small"
 			(at 247.65 137.0965 0)
@@
 			)
 		)
+		(property "MPN" "L-53SGC"
+			(at 107.696 135.89 0)
+			(hide yes)
+			(show_name no)
+			(do_not_autoplace no)
+			(effects
+				(font
+					(size 1.27 1.27)
+				)
+			)
+		)
 		(property "Value" "LED_Small"
 			(at 109.22 135.8265 0)
@@
 			)
 		)
+		(property "MPN" "L-53SGC"
+			(at 233.426 137.16 0)
+			(hide yes)
+			(show_name no)
+			(do_not_autoplace no)
+			(effects
+				(font
+					(size 1.27 1.27)
+				)
+			)
+		)
 		(property "Value" "LED_Small"
 			(at 234.95 137.0965 0)
@@
 			)
 		)
+		(property "MPN" "L-53SGC"
+			(at 235.966 137.16 0)
+			(hide yes)
+			(show_name no)
+			(do_not_autoplace no)
+			(effects
+				(font
+					(size 1.27 1.27)
+				)
+			)
+		)
 		(property "Value" "LED_Small"
 			(at 237.49 137.0965 0)
@@
 			)
 		)
+		(property "MPN" "L-53SGC"
+			(at 110.236 135.89 0)
+			(hide yes)
+			(show_name no)
+			(do_not_autoplace no)
+			(effects
+				(font
+					(size 1.27 1.27)
+				)
+			)
+		)
 		(property "Value" "LED_Small"
 			(at 111.76 135.8265 0)
@@
 			)
 		)
+		(property "MPN" "L-53SGC"
+			(at 97.536 135.89 0)
+			(hide yes)
+			(show_name no)
+			(do_not_autoplace no)
+			(effects
+				(font
+					(size 1.27 1.27)
+				)
+			)
+		)
 		(property "Value" "LED_Small"
 			(at 99.06 135.8265 0)
@@
 			)
 		)
+		(property "MPN" "L-53SGC"
+			(at 112.776 135.89 0)
+			(hide yes)
+			(show_name no)
+			(do_not_autoplace no)
+			(effects
+				(font
+					(size 1.27 1.27)
+				)
+			)
+		)
 		(property "Value" "LED_Small"
 			(at 114.3 135.8265 0)
@@
 			)
 		)
+		(property "MPN" "L-53SGC"
+			(at 115.316 135.89 0)
+			(hide yes)
+			(show_name no)
+			(do_not_autoplace no)
+			(effects
+				(font
+					(size 1.27 1.27)
+				)
+			)
+		)
 		(property "Value" "LED_Small"
 			(at 116.84 135.8265 0)
@@
 			)
 		)
+		(property "MPN" "L-53SGC"
+			(at 248.666 137.16 0)
+			(hide yes)
+			(show_name no)
+			(do_not_autoplace no)
+			(effects
+				(font
+					(size 1.27 1.27)
+				)
+			)
+		)
 		(property "Value" "LED_Small"
 			(at 250.19 137.0965 0)
@@
 			)
 		)
+		(property "MPN" "L-53SGC"
+			(at 230.886 137.16 0)
+			(hide yes)
+			(show_name no)
+			(do_not_autoplace no)
+			(effects
+				(font
+					(size 1.27 1.27)
+				)
+			)
+		)
 		(property "Value" "LED_Small"
 			(at 232.41 137.0965 0)
@@
 			)
 		)
+		(property "MPN" "L-53SGC"
+			(at 100.076 135.89 0)
+			(hide yes)
+			(show_name no)
+			(do_not_autoplace no)
+			(effects
+				(font
+					(size 1.27 1.27)
+				)
+			)
+		)
 		(property "Value" "LED_Small"
 			(at 101.6 135.8265 0)
@@
 			(at 102.616 135.89 0)
 			(hide yes)
+			(show_name no)
+			(do_not_autoplace no)
+			(effects
+				(font
+					(size 1.27 1.27)
+				)
+			)
+		)
+		(property "MPN" "L-53SGC"
+			(at 102.616 135.89 0)
+			(hide yes)

Commit message: Standardise LEDs on Supplier Ref (Element14-only sourcing)
Only Element14 is used for LEDs, so identify every LED by its
Element14 Supplier Ref and carry no MPN on LEDs. Move the green LEDs'
L-53SGC from MPN to Supplier Ref (red 703-0100 already there). MPN
stays reserved for the socketed chips (manufacturer parts). Update the
LED sourcing table in CLAUDE.md.

Co-Authored-By: Claude Opus 4.8 (1M context) <noreply@anthropic.com>
Parts:
- D20, D21, D22, D23, D24, D25, D26, D27, D28, D29, D30, D31, D32, D33, D34, D35: MPN L-53SGC -> (none); Supplier Ref (none) -> L-53SGC
Changed lines of the file:
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@@
 			)
 		)
-		(property "MPN" "L-53SGC"
+		(property "Supplier Ref" "L-53SGC"
 			(at 105.156 135.89 0)
 			(hide yes)
@@
 			)
 		)
-		(property "MPN" "L-53SGC"
+		(property "Supplier Ref" "L-53SGC"
 			(at 238.506 137.16 0)
 			(hide yes)
@@
 			)
 		)
-		(property "MPN" "L-53SGC"
+		(property "Supplier Ref" "L-53SGC"
 			(at 241.046 137.16 0)
 			(hide yes)
@@
 			)
 		)
-		(property "MPN" "L-53SGC"
+		(property "Supplier Ref" "L-53SGC"
 			(at 243.586 137.16 0)
 			(hide yes)
@@
 			)
 		)
-		(property "MPN" "L-53SGC"
+		(property "Supplier Ref" "L-53SGC"
 			(at 246.126 137.16 0)
 			(hide yes)
@@
 			)
 		)
-		(property "MPN" "L-53SGC"
+		(property "Supplier Ref" "L-53SGC"
 			(at 107.696 135.89 0)
 			(hide yes)
@@
 			)
 		)
-		(property "MPN" "L-53SGC"
+		(property "Supplier Ref" "L-53SGC"
 			(at 233.426 137.16 0)
 			(hide yes)
@@
 			)
 		)
-		(property "MPN" "L-53SGC"
+		(property "Supplier Ref" "L-53SGC"
 			(at 235.966 137.16 0)
 			(hide yes)
@@
 			)
 		)
-		(property "MPN" "L-53SGC"
+		(property "Supplier Ref" "L-53SGC"
 			(at 110.236 135.89 0)
 			(hide yes)
@@
 			)
 		)
-		(property "MPN" "L-53SGC"
+		(property "Supplier Ref" "L-53SGC"
 			(at 97.536 135.89 0)
 			(hide yes)
@@
 			)
 		)
-		(property "MPN" "L-53SGC"
+		(property "Supplier Ref" "L-53SGC"
 			(at 112.776 135.89 0)
 			(hide yes)
@@
 			)
 		)
-		(property "MPN" "L-53SGC"
+		(property "Supplier Ref" "L-53SGC"
 			(at 115.316 135.89 0)
 			(hide yes)
@@
 			)
 		)
-		(property "MPN" "L-53SGC"
+		(property "Supplier Ref" "L-53SGC"
 			(at 248.666 137.16 0)
 			(hide yes)
@@
 			)
 		)
-		(property "MPN" "L-53SGC"
+		(property "Supplier Ref" "L-53SGC"
 			(at 230.886 137.16 0)
 			(hide yes)
@@
 			)
 		)
-		(property "MPN" "L-53SGC"
+		(property "Supplier Ref" "L-53SGC"
 			(at 100.076 135.89 0)
 			(hide yes)
@@
 			)
 		)
-		(property "MPN" "L-53SGC"
+		(property "Supplier Ref" "L-53SGC"
 			(at 102.616 135.89 0)
 			(hide yes)

Commit message: Tag yellow LEDs with Element14 Supplier Ref MCL053YD
Add Supplier Ref MCL053YD to the 11 yellow front-panel LEDs and update
the LED sourcing table in CLAUDE.md. White and blue still uncoded.

Co-Authored-By: Claude Opus 4.8 (1M context) <noreply@anthropic.com>
Parts:
- D79, D84: Supplier Ref (none) -> MCL053YD
Changed lines of the file:
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@@
+			)
+		)
+		(property "Supplier Ref" "MCL053YD"
+			(at 184.404 137.16 0)
+			(hide yes)
+			(show_name no)
+			(do_not_autoplace no)
+			(effects
+				(font
+					(size 1.27 1.27)
+				)
 			)
 		)
@@
 			(at 161.544 137.16 0)
 			(hide yes)
+			(show_name no)
+			(do_not_autoplace no)
+			(effects
+				(font
+					(size 1.27 1.27)
+				)
+			)
+		)
+		(property "Supplier Ref" "MCL053YD"
+			(at 161.544 137.16 0)
+			(hide yes)

Commit message: Tag white LEDs with Element14 Supplier Ref C512A-WNN-CZ0B0151
Add Supplier Ref C512A-WNN-CZ0B0151 to the 4 white front-panel LEDs
and update the LED sourcing table in CLAUDE.md. Only blue left.

Co-Authored-By: Claude Opus 4.8 (1M context) <noreply@anthropic.com>
Parts:
- D92: Supplier Ref (none) -> C512A-WNN-CZ0B0151
Changed lines of the file:
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@@
+			)
+		)
+		(property "Supplier Ref" "C512A-WNN-CZ0B0151"
+			(at 173.736 137.16 0)
+			(hide yes)
+			(show_name no)
+			(do_not_autoplace no)
+			(effects
+				(font
+					(size 1.27 1.27)
+				)
 			)
 		)
