File: KiCAD10/PC.kicad_sch (KiCad schematic)
At the start: 34 parts, among them U24 74HC245, U25 74HC161, U26 74HC161, U27 74HC245, U28 74HC161, U29 74HC161

Commit message: Fix red LED Supplier Ref: use Element14 order code 2112111
703-0100 was the Multicomp MPN, not an Element14 order code. All 7
red LEDs (AO BO EO TO COH COL RO) now carry the numeric code, and
the CLAUDE.md sourcing table matches.

Co-Authored-By: Claude Fable 5 <noreply@anthropic.com>
Parts:
- D81, D83: Supplier Ref 703-0100 -> 2112111
Changed lines of the file:
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@@
 			)
 		)
-		(property "Supplier Ref" "703-0100"
+		(property "Supplier Ref" "2112111"
 			(at 176.784 137.16 0)
 			(hide yes)
@@
 			)
 		)
-		(property "Supplier Ref" "703-0100"
+		(property "Supplier Ref" "2112111"
 			(at 153.924 137.16 0)
 			(hide yes)
