File: KiCAD10/ALU.kicad_sch (KiCad schematic)
At the start: 23 parts, among them U13 74HC283, U30 74HC86, U31 74HC86, U32 74HC4002, U33 74HC283, U34 74HC245

Commit message: Capture as-built LED colours as schematic Color field
Prepping the BOM/PCB for a prototype fab run: the front-panel LED
colour was only recorded per-footprint on the PCB (the Description
field, e.g. "LED GREEN, 2000mcd, 60°") and so never reached the
schematic-generated BOM. Copy that colour onto all 98 LED symbols as
a hidden `Color` property, matched by reference designator, so it
travels with the BOM the same way `MPN` does (add `Color` to the BOM
export field list). As-built distribution: Green 75, Yellow 11,
Red 7, White 4, Blue 1.

Source of truth for colour is now the schematic `Color` field; the
PCB footprint `Description` is the independent original and KiCad does
not auto-sync the two.

Also folds in KiCad 10 file normalisation that appeared on opening the
project (new .kicad_pro design-setting defaults; empty "element"
properties added to symbols on the top sheet). Document all of the
above in CLAUDE.md.

Co-Authored-By: Claude Opus 4.8 (1M context) <noreply@anthropic.com>
Parts:
- D52, D53, D54, D55, D56, D57, D58: Color (none) -> Green; element14 (none) -> 1003234
- D59, D95: Color (none) -> Green
- D78: Color (none) -> Red
- D93, D94: Color (none) -> White

Commit message: Tag red LEDs with Element14 order code 703-0100
Add MPN 703-0100 to the 7 red front-panel LEDs (D66 AO, D77 BO,
D78 EO, D80 TO, D81 COH, D83 COL, D99 RO) for the Element14 order.

Co-Authored-By: Claude Opus 4.8 (1M context) <noreply@anthropic.com>
Parts:
- D78: MPN (none) -> 703-0100
Changed lines of the file:
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@@
+			)
+		)
+		(property "MPN" "703-0100"
+			(at 134.874 170.18 0)
+			(hide yes)
+			(show_name no)
+			(do_not_autoplace no)
+			(effects
+				(font
+					(size 1.27 1.27)
+				)
 			)
 		)

Commit message: Move LED Element14 code from MPN to Supplier Ref field
Element14/Farnell order codes are distributor codes, not manufacturer
part numbers, so keep them out of MPN (which holds manufacturer PNs
like SST39SF010A-70-4C-PHE for the chips). Migrate the red LEDs'
703-0100 into a dedicated 'Supplier Ref' property and document the
MPN vs Supplier Ref convention in CLAUDE.md.

Co-Authored-By: Claude Opus 4.8 (1M context) <noreply@anthropic.com>
Parts:
- D78: MPN 703-0100 -> (none); Supplier Ref (none) -> 703-0100
Changed lines of the file:
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@@
 			)
 		)
-		(property "MPN" "703-0100"
+		(property "Supplier Ref" "703-0100"
 			(at 134.874 170.18 0)
 			(hide yes)

Commit message: Tag green LEDs with Kingbright MPN L-53SGC
Green LED part is Kingbright L-53SGC — a manufacturer part number, so
it goes in MPN (all 75 green LEDs), unlike the red LEDs' Farnell code
which lives in Supplier Ref. Update the LED sourcing table in CLAUDE.md.

Co-Authored-By: Claude Opus 4.8 (1M context) <noreply@anthropic.com>
Parts:
- D52, D53, D54, D55, D56, D57, D58, D59, D95: MPN (none) -> L-53SGC
Changed lines of the file:
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@@
+			)
+		)
+		(property "MPN" "L-53SGC"
+			(at 81.026 121.92 0)
+			(hide yes)
+			(show_name no)
+			(do_not_autoplace no)
+			(effects
+				(font
+					(size 1.27 1.27)
+				)
 			)
 		)
@@
 			)
 		)
+		(property "MPN" "L-53SGC"
+			(at 78.486 121.92 0)
+			(hide yes)
+			(show_name no)
+			(do_not_autoplace no)
+			(effects
+				(font
+					(size 1.27 1.27)
+				)
+			)
+		)
 		(property "Value" "LED_Small"
 			(at 80.01 121.8565 0)
@@
 			)
 		)
+		(property "MPN" "L-53SGC"
+			(at 88.646 121.92 0)
+			(hide yes)
+			(show_name no)
+			(do_not_autoplace no)
+			(effects
+				(font
+					(size 1.27 1.27)
+				)
+			)
+		)
 		(property "Value" "LED_Small"
 			(at 90.17 121.8565 0)
@@
 		)
 		(property "Color" "Green"
+			(at 83.566 121.92 0)
+			(hide yes)
+			(show_name no)
+			(do_not_autoplace no)
+			(effects
+				(font
+					(size 1.27 1.27)
+				)
+			)
+		)
+		(property "MPN" "L-53SGC"
 			(at 83.566 121.92 0)
 			(hide yes)
@@
 			)
 		)
+		(property "MPN" "L-53SGC"
+			(at 86.106 121.92 0)
+			(hide yes)
+			(show_name no)
+			(do_not_autoplace no)
+			(effects
+				(font
+					(size 1.27 1.27)
+				)
+			)
+		)
 		(property "Value" "LED_Small"
 			(at 87.63 121.8565 0)
@@
 			)
 		)
+		(property "MPN" "L-53SGC"
+			(at 194.056 118.11 0)
+			(hide yes)
+			(show_name no)
+			(do_not_autoplace no)
+			(effects
+				(font
+					(size 1.27 1.27)
+				)
+			)
+		)
 		(property "Value" "C"
 			(at 188.976 118.364 0)
@@
 		)
 		(property "Color" "Green"
+			(at 75.946 121.92 0)
+			(hide yes)
+			(show_name no)
+			(do_not_autoplace no)
+			(effects
+				(font
+					(size 1.27 1.27)
+				)
+			)
+		)
+		(property "MPN" "L-53SGC"
 			(at 75.946 121.92 0)
 			(hide yes)
@@
 			)
 		)
+		(property "MPN" "L-53SGC"
+			(at 73.406 121.92 0)
+			(hide yes)
+			(show_name no)
+			(do_not_autoplace no)
+			(effects
+				(font
+					(size 1.27 1.27)
+				)
+			)
+		)
 		(property "Value" "LED_Small"
 			(at 74.93 121.8565 0)
@@
 			(at 91.186 121.92 0)
 			(hide yes)
+			(show_name no)
+			(do_not_autoplace no)
+			(effects
+				(font
+					(size 1.27 1.27)
+				)
+			)
+		)
+		(property "MPN" "L-53SGC"
+			(at 91.186 121.92 0)
+			(hide yes)

Commit message: Standardise LEDs on Supplier Ref (Element14-only sourcing)
Only Element14 is used for LEDs, so identify every LED by its
Element14 Supplier Ref and carry no MPN on LEDs. Move the green LEDs'
L-53SGC from MPN to Supplier Ref (red 703-0100 already there). MPN
stays reserved for the socketed chips (manufacturer parts). Update the
LED sourcing table in CLAUDE.md.

Co-Authored-By: Claude Opus 4.8 (1M context) <noreply@anthropic.com>
Parts:
- D52, D53, D54, D55, D56, D57, D58, D59, D95: MPN L-53SGC -> (none); Supplier Ref (none) -> L-53SGC
Changed lines of the file:
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@@
 			)
 		)
-		(property "MPN" "L-53SGC"
+		(property "Supplier Ref" "L-53SGC"
 			(at 81.026 121.92 0)
 			(hide yes)
@@
 			)
 		)
-		(property "MPN" "L-53SGC"
+		(property "Supplier Ref" "L-53SGC"
 			(at 78.486 121.92 0)
 			(hide yes)
@@
 			)
 		)
-		(property "MPN" "L-53SGC"
+		(property "Supplier Ref" "L-53SGC"
 			(at 88.646 121.92 0)
 			(hide yes)
@@
 			)
 		)
-		(property "MPN" "L-53SGC"
+		(property "Supplier Ref" "L-53SGC"
 			(at 83.566 121.92 0)
 			(hide yes)
@@
 			)
 		)
-		(property "MPN" "L-53SGC"
+		(property "Supplier Ref" "L-53SGC"
 			(at 86.106 121.92 0)
 			(hide yes)
@@
 			)
 		)
-		(property "MPN" "L-53SGC"
+		(property "Supplier Ref" "L-53SGC"
 			(at 194.056 118.11 0)
 			(hide yes)
@@
 			)
 		)
-		(property "MPN" "L-53SGC"
+		(property "Supplier Ref" "L-53SGC"
 			(at 75.946 121.92 0)
 			(hide yes)
@@
 			)
 		)
-		(property "MPN" "L-53SGC"
+		(property "Supplier Ref" "L-53SGC"
 			(at 73.406 121.92 0)
 			(hide yes)
@@
 			)
 		)
-		(property "MPN" "L-53SGC"
+		(property "Supplier Ref" "L-53SGC"
 			(at 91.186 121.92 0)
 			(hide yes)

Commit message: Tag white LEDs with Element14 Supplier Ref C512A-WNN-CZ0B0151
Add Supplier Ref C512A-WNN-CZ0B0151 to the 4 white front-panel LEDs
and update the LED sourcing table in CLAUDE.md. Only blue left.

Co-Authored-By: Claude Opus 4.8 (1M context) <noreply@anthropic.com>
Parts:
- D93, D94: Supplier Ref (none) -> C512A-WNN-CZ0B0151
Changed lines of the file:
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@@
+			)
+		)
+		(property "Supplier Ref" "C512A-WNN-CZ0B0151"
+			(at 91.186 88.9 0)
+			(hide yes)
+			(show_name no)
+			(do_not_autoplace no)
+			(effects
+				(font
+					(size 1.27 1.27)
+				)
 			)
 		)
@@
 			(at 192.786 53.34 0)
 			(hide yes)
+			(show_name no)
+			(do_not_autoplace no)
+			(effects
+				(font
+					(size 1.27 1.27)
+				)
+			)
+		)
+		(property "Supplier Ref" "C512A-WNN-CZ0B0151"
+			(at 192.786 53.34 0)
+			(hide yes)

Commit message: Fix red LED Supplier Ref: use Element14 order code 2112111
703-0100 was the Multicomp MPN, not an Element14 order code. All 7
red LEDs (AO BO EO TO COH COL RO) now carry the numeric code, and
the CLAUDE.md sourcing table matches.

Co-Authored-By: Claude Fable 5 <noreply@anthropic.com>
Parts:
- D78: Supplier Ref 703-0100 -> 2112111
Changed lines of the file:
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@@
 			)
 		)
-		(property "Supplier Ref" "703-0100"
+		(property "Supplier Ref" "2112111"
 			(at 134.874 170.18 0)
 			(hide yes)
