File: KiCAD10/UART_RX.kicad_sch (KiCad schematic)
At the start: 11 parts, among them J1 UART, U1 74HC00, U2 74HC193, U3 74HC161, U4 74HC595, U5 74HC165

Commit message: Capture as-built LED colours as schematic Color field
Prepping the BOM/PCB for a prototype fab run: the front-panel LED
colour was only recorded per-footprint on the PCB (the Description
field, e.g. "LED GREEN, 2000mcd, 60°") and so never reached the
schematic-generated BOM. Copy that colour onto all 98 LED symbols as
a hidden `Color` property, matched by reference designator, so it
travels with the BOM the same way `MPN` does (add `Color` to the BOM
export field list). As-built distribution: Green 75, Yellow 11,
Red 7, White 4, Blue 1.

Source of truth for colour is now the schematic `Color` field; the
PCB footprint `Description` is the independent original and KiCad does
not auto-sync the two.

Also folds in KiCad 10 file normalisation that appeared on opening the
project (new .kicad_pro design-setting defaults; empty "element"
properties added to symbols on the top sheet). Document all of the
above in CLAUDE.md.

Co-Authored-By: Claude Opus 4.8 (1M context) <noreply@anthropic.com>
Parts:
- D80: Color (none) -> Red
- D97: Color (none) -> Blue
Changed lines of the file:
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@@
 			)
 		)
+		(property "element14" ""
+			(at 104.14 106.68 0)
+			(hide yes)
+			(show_name no)
+			(do_not_autoplace no)
+			(effects
+				(font
+					(size 1.27 1.27)
+				)
+			)
+		)
 		(pin "1"
 		)
@@
 			)
 		)
+		(property "element14" ""
+			(at 104.14 93.98 0)
+			(hide yes)
+			(show_name no)
+			(do_not_autoplace no)
+			(effects
+				(font
+					(size 1.27 1.27)
+				)
+			)
+		)
 		(pin "1"
 		)
@@
 			)
 		)
+		(property "element14" ""
+			(at 88.9 91.44 0)
+			(hide yes)
+			(show_name no)
+			(do_not_autoplace no)
+			(effects
+				(font
+					(size 1.27 1.27)
+				)
+			)
+		)
 		(pin "1"
 		)
@@
 			)
 		)
+		(property "element14" ""
+			(at 119.38 152.4 90)
+			(hide yes)
+			(show_name no)
+			(do_not_autoplace no)
+			(effects
+				(font
+					(size 1.27 1.27)
+				)
+			)
+		)
 		(pin "1"
 		)
@@
 			)
 		)
+		(property "element14" ""
+			(at 77.47 88.9 90)
+			(hide yes)
+			(show_name no)
+			(do_not_autoplace no)
+			(effects
+				(font
+					(size 1.27 1.27)
+				)
+			)
+		)
 		(pin "1"
 		)
@@
 			)
 		)
+		(property "element14" ""
+			(at 73.66 129.54 0)
+			(hide yes)
+			(show_name no)
+			(do_not_autoplace no)
+			(effects
+				(font
+					(size 1.27 1.27)
+				)
+			)
+		)
 		(pin "1"
 		)
@@
 			)
 		)
+		(property "element14" ""
+			(at 185.42 76.2 90)
+			(hide yes)
+			(show_name no)
+			(do_not_autoplace no)
+			(effects
+				(font
+					(size 1.27 1.27)
+				)
+			)
+		)
 		(pin "1"
 		)
@@
 			)
 		)
+		(property "element14" ""
+			(at 74.93 68.58 90)
+			(hide yes)
+			(show_name no)
+			(do_not_autoplace no)
+			(effects
+				(font
+					(size 1.27 1.27)
+				)
+			)
+		)
 		(pin "1"
 		)
@@
 			)
 		)
+		(property "Color" "Blue"
+			(at 124.714 146.05 0)
+			(hide yes)
+			(show_name no)
+			(do_not_autoplace no)
+			(effects
+				(font
+					(size 1.27 1.27)
+				)
+			)
+		)
 		(property "Value" "R"
 			(at 124.968 146.05 0)
@@
 			)
 		)
+		(property "element14" ""
+			(at 127 146.05 0)
+			(hide yes)
+			(show_name no)
+			(do_not_autoplace no)
+			(effects
+				(font
+					(size 1.27 1.27)
+				)
+			)
+		)
 		(pin "2"
 		)
@@
 			)
 		)
+		(property "element14" ""
+			(at 170.18 115.57 90)
+			(hide yes)
+			(show_name no)
+			(do_not_autoplace no)
+			(effects
+				(font
+					(size 1.27 1.27)
+				)
+			)
+		)
 		(pin "1"
 		)
@@
 			)
 		)
+		(property "element14" ""
+			(at 129.54 115.57 90)
+			(hide yes)
+			(show_name no)
+			(do_not_autoplace no)
+			(effects
+				(font
+					(size 1.27 1.27)
+				)
+			)
+		)
 		(pin "1"
 		)
@@
 			)
 		)
+		(property "element14" ""
+			(at 134.62 76.2 90)
+			(hide yes)
+			(show_name no)
+			(do_not_autoplace no)
+			(effects
+				(font
+					(size 1.27 1.27)
+				)
+			)
+		)
 		(pin "1"
 		)
@@
 			)
 		)
+		(property "Color" "Red"
+			(at 117.094 146.05 0)
+			(hide yes)
+			(show_name no)
+			(do_not_autoplace no)
+			(effects
+				(font
+					(size 1.27 1.27)
+				)
+			)
+		)
 		(property "Value" "TO"
 			(at 117.094 146.05 0)
@@
 			)
 		)
+		(property "element14" ""
+			(at 119.38 146.05 0)
+			(hide yes)
+			(show_name no)
+			(do_not_autoplace no)
+			(effects
+				(font
+					(size 1.27 1.27)
+				)
+			)
+		)
 		(pin "2"
 		)
@@
 			)
 		)
+		(property "element14" ""
+			(at 66.04 88.9 0)
+			(hide yes)
+			(show_name no)
+			(do_not_autoplace no)
+			(effects
+				(font
+					(size 1.27 1.27)
+				)
+			)
+		)
 		(pin "1"
 		)
@@
 			(hide yes)
 			(show_name no)
+			(do_not_autoplace no)
+			(effects
+				(font
+					(size 1.27 1.27)
+				)
+			)
+		)
+		(property "element14" ""
+			(at 127 152.4 90)
+			(hide yes)
+			(show_name no)

Commit message: Tag red LEDs with Element14 order code 703-0100
Add MPN 703-0100 to the 7 red front-panel LEDs (D66 AO, D77 BO,
D78 EO, D80 TO, D81 COH, D83 COL, D99 RO) for the Element14 order.

Co-Authored-By: Claude Opus 4.8 (1M context) <noreply@anthropic.com>
Parts:
- D80: MPN (none) -> 703-0100
Changed lines of the file:
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@@
+			)
+		)
+		(property "MPN" "703-0100"
+			(at 117.094 146.05 0)
+			(hide yes)
+			(show_name no)
+			(do_not_autoplace no)
+			(effects
+				(font
+					(size 1.27 1.27)
+				)
 			)
 		)

Commit message: Move LED Element14 code from MPN to Supplier Ref field
Element14/Farnell order codes are distributor codes, not manufacturer
part numbers, so keep them out of MPN (which holds manufacturer PNs
like SST39SF010A-70-4C-PHE for the chips). Migrate the red LEDs'
703-0100 into a dedicated 'Supplier Ref' property and document the
MPN vs Supplier Ref convention in CLAUDE.md.

Co-Authored-By: Claude Opus 4.8 (1M context) <noreply@anthropic.com>
Parts:
- D80: MPN 703-0100 -> (none); Supplier Ref (none) -> 703-0100
Changed lines of the file:
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@@
 			)
 		)
-		(property "MPN" "703-0100"
+		(property "Supplier Ref" "703-0100"
 			(at 117.094 146.05 0)
 			(hide yes)

Commit message: Tag blue LED with Element14 Supplier Ref C503B-BCS-CV0Z0461
Add Supplier Ref C503B-BCS-CV0Z0461 to the single blue LED (D97). All
98 front-panel LEDs are now coded for Element14; update the CLAUDE.md
sourcing table.

Co-Authored-By: Claude Opus 4.8 (1M context) <noreply@anthropic.com>
Parts:
- D97: Supplier Ref (none) -> C503B-BCS-CV0Z0461
Changed lines of the file:
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@@
+			)
+		)
+		(property "Supplier Ref" "C503B-BCS-CV0Z0461"
+			(at 124.714 146.05 0)
+			(hide yes)
+			(show_name no)
+			(do_not_autoplace no)
+			(effects
+				(font
+					(size 1.27 1.27)
+				)
 			)
 		)

Commit message: Fix red LED Supplier Ref: use Element14 order code 2112111
703-0100 was the Multicomp MPN, not an Element14 order code. All 7
red LEDs (AO BO EO TO COH COL RO) now carry the numeric code, and
the CLAUDE.md sourcing table matches.

Co-Authored-By: Claude Fable 5 <noreply@anthropic.com>
Parts:
- D80: Supplier Ref 703-0100 -> 2112111
Changed lines of the file:
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@@
 			)
 		)
-		(property "Supplier Ref" "703-0100"
+		(property "Supplier Ref" "2112111"
 			(at 117.094 146.05 0)
 			(hide yes)
